Commit message: changes to collision constrains supressing torque and velocity constrains and adding model measurment files

File: model/try1.urdf (robot description, URDF)
Before this commit: robot youbot, 7 links, 6 joints
Joints:
- joint arm_joint_1: origin xyz=0.024 0 0.096 rpy=0 0 2.96705972839 -> xyz=0.0 0 0.0 rpy=0 0 2.96705972839
- joint arm_joint_2: origin xyz=0.033 0 0.019 rpy=0 -1.1344640138 0 -> xyz=0.0 0 0.5 rpy=0 -1.1344640138 0
- joint arm_joint_3: origin xyz=0.000 0.000 0.155 rpy=0 2.54818070791 0 -> xyz=0.000 0.000 0.555 rpy=0 2.54818070791 0
- joint arm_joint_4: origin xyz=0.000 0.000 0.135 rpy=0 -1.78896248329 0 -> xyz=0.000 0.000 0.535 rpy=0 -1.78896248329 0
- joint arm_joint_5: axis 0 0 -1 -> 0 0 1; origin xyz=-0.002 0 0.130 rpy=0 0 2.92342649709 -> xyz=0.0 0 0.530 rpy=0 0 2.92342649709

File: model/try2.urdf (robot description, URDF)
Before this commit: robot youbot, 7 links, 6 joints
Links:
- removed link arm_link_4
- removed link arm_link_5
Joints:
- removed joint arm_joint_4
- removed joint arm_joint_5
